File: cape/uCAN Cape.brd (EAGLE design)
At the start: 71.8 x 54.6 mm, 21 parts, among them CN1 RJ45-8PTH, CN2 RJ45-8PTH, IC1 LM2592HVS-5.0, IC2 MCP2562, IC3 EEPROM-I2CSMD

Commit message: Minor changes to shield, rpi board, and cape
Parts:
- removed C1: 4.7u, SparkFun-Capacitors:1206
- removed C2: 47u, SparkFun-Capacitors:PANASONIC_C
- removed L1: MSS1260, nickparts:MSS1260
- added C10: 56u, nickparts:SM_RADIAL_6.3AMM
- added C3: 4.7u, nickparts:1206
- added C4: 1u, nickparts:0805
- added C9: 10n, nickparts:0805
- added I1: SRN8040-330M, nickparts:SRN8040
- D1: value (none) -> B240A-13-F; device SparkFun-DiscreteSemi:SMA-DIODE_ALT -> nickparts:SMA
- IC1: value LM2592HVS-5.0 -> LM22675MR-5.0/NOPB; device nickparts:TO263-5 -> nickparts:MRA08B
- moved D1 22.8 mm to (49.2, 34.9)
- moved IC1 8.64 mm to (41.3, 34.3)
Connections:
- removed net N$11: CN1.5, CN2.5
- new net N$9: CN1.3, CN2.3
- net GND: now also C10.2, C3.2, C4.2, CN1.8, CN2.8, D1.2, IC1.EPAD; no longer C1.2, C2.-, CN1.3, CN2.3, D1.A, IC1.3, IC1.5
- net N$10: now also C9.1, IC1.1; no longer CN1.4, CN2.4
- net SWOUT: now also C9.2, D1.1, I1.2, IC1.8; no longer D1.C, IC1.1, L1.P$1
- net V+: now also C10.1, I1.1; no longer C2.+, L1.P$2
- net VCC: now also C3.1, C4.1, CN1.4, CN1.5, CN2.4, CN2.5, IC1.7; no longer C1.1, CN1.8, CN2.8, IC1.2
Routing:
- net GND: track 325.2 -> 256.2 mm, vias 59 -> 15
- net N$10: track 26.2 -> 2.62 mm, vias 1 -> 0
- net N$11: track 22.4 -> 0.00 mm, vias 1 -> 0
- net N$9: track 0.00 -> 21.2 mm, vias 0 -> 1
- net N$12: track 38.9 -> 27.5 mm
- net V+: track 93.3 -> 82.6 mm
- net VCC: track 32.4 -> 38.1 mm
- net SWOUT: track 20.3 -> 17.6 mm
- removed copper zone on layer 1, net VCC
Other:
- board text added: "uCAN Cape v0.1.1"
- board text removed: "uCAN Cape v0.1"
