File: cape/uCAN Cape.sch (EAGLE design)
At the start: 19 parts, among them CN1 RJ45-8PTH, CN2 RJ45-8PTH, IC1 LM2592HVS-5.0, IC2 MCP2562, IC3 EEPROM-I2CSMD

Commit message: Minor changes to shield, rpi board, and cape
Parts:
- removed C1: 4.7u, SparkFun-Capacitors:CAP1206
- removed C2: 47u, SparkFun-Capacitors:CAP_POLC
- removed L1: MSS1260, nickparts:MSS1260
- added C10: 56u, nickparts:10SVP56M
- added C3: 4.7u, nickparts:GRM31CR71H475KA12L
- added C4: 1u, nickparts:GMK212B7105KG-T
- added C9: 10n, nickparts:C0805C103K5RACTU
- added I1: SRN8040-330M, nickparts:SRN8040-330M
- D1: value (none) -> B240A-13-F; device SparkFun-DiscreteSemi:DIODESMA-ALT -> nickparts:B240A-13-F
- IC1: value LM2592HVS-5.0 -> LM22675MR-5.0/NOPB; device nickparts:LM2595NDH -> nickparts:LM22675MR-5.0/NOPB
Connections:
- removed net N$11: CN1.5, CN2.5
- new net N$9: CN1.3, CN2.3
- net GND: now also C10.-, C3.2, C4.2, CN1.8, CN2.8; no longer C1.2, C2.-, CN1.3, CN2.3, IC1./EN
- net N$10: now also C9.1, IC1.BOOT; no longer CN1.4, CN2.4
- net SWOUT: now also C9.2, D1.K, I1.2, IC1.SW; no longer D1.C, IC1.OUT, L1.1
- net V+: now also C10.+, I1.1; no longer C2.+, L1.2
- net VCC: now also C3.1, C4.1, CN1.4, CN1.5, CN2.4, CN2.5; no longer C1.1, CN1.8, CN2.8
