File: injector/injector.brd (EAGLE design)
At the start: 39 x 15.2 mm, 6 parts, among them J1 POWER_JACKPTH

Commit message: Minor changes to shield, rpi board, and cape
Parts:
- moved C1 4.45 mm to (19.7, 11.4)
- moved J1 4.45 mm to (36.2, 7.62)
- moved R1 4.45 mm to (17.8, 14.0)
- moved R2 4.45 mm to (17.8, 8.89)
- moved U$1 4.45 mm to (5.71, 7.62)
Connections:
- net N$3: now also U$1.4, U$1.5; no longer U$1.8
- net N$4: now also U$1.8
Routing:
- net N$4: track 33.0 -> 29.6 mm
- net N$3: track 9.73 -> 11.2 mm
Other:
- board size 39 x 15.2 mm -> 34.6 x 15.2 mm
- board text added: "uCAN Power Injector v1.0.1"
- board text removed: "uCAN Power Injector v1.0"
Changed lines of the file:
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@@
 <board>
 <plain>
-<wire x1="0" y1="0" x2="39.04" y2="0" width="0" layer="20"/>
-<wire x1="39.04" y1="0" x2="39.04" y2="15.23" width="0" layer="20"/>
-<wire x1="39.04" y1="15.23" x2="0" y2="15.23" width="0" layer="20"/>
+<wire x1="0" y1="0" x2="34.595" y2="0" width="0" layer="20"/>
+<wire x1="34.595" y1="0" x2="34.595" y2="15.23" width="0" layer="20"/>
+<wire x1="34.595" y1="15.23" x2="0" y2="15.23" width="0" layer="20"/>
 <wire x1="0" y1="15.23" x2="0" y2="0" width="0" layer="20"/>
-<text x="13.97" y="7.62" size="0.889" layer="26" font="vector" ratio="17" rot="MR270" align="bottom-center">uCAN Power Injector
-v1.0</text>
+<text x="33.655" y="7.62" size="0.889" layer="26" font="vector" ratio="17" rot="MR270" align="bottom-center">uCAN Power Injector
+v1.0.1</text>
 </plain>
 <attributes>
@@
 </autorouter>
 <elements>
-<element name="U$1" library="SparkFun-Connectors" package="RJ45-8" value="RJ45-8PTH" x="10.16" y="7.62" rot="R270"/>
-<element name="R1" library="SparkFun-Passives" package="0603-RES" value="60" x="22.225" y="13.97" smashed="yes">
-<attribute name="NAME" x="23.876" y="13.462" size="1.016" layer="25" font="vector" ratio="15"/>
-</element>
-<element name="J1" library="SparkFun-Connectors" package="POWER_JACK_PTH" value="POWER_JACKPTH" x="40.64" y="7.62" smashed="yes" rot="R90">
-<attribute name="NAME" x="35.56" y="3.81" size="1.016" layer="25" font="vector" ratio="15" rot="R90"/>
+<element name="U$1" library="SparkFun-Connectors" package="RJ45-8" value="RJ45-8PTH" x="5.715" y="7.62" rot="R270"/>
+<element name="R1" library="SparkFun-Passives" package="0603-RES" value="60" x="17.78" y="13.97" smashed="yes">
+<attribute name="NAME" x="19.431" y="13.462" size="1.016" layer="25" font="vector" ratio="15"/>
+</element>
+<element name="J1" library="SparkFun-Connectors" package="POWER_JACK_PTH" value="POWER_JACKPTH" x="36.195" y="7.62" smashed="yes" rot="R90">
+<attribute name="NAME" x="31.115" y="3.81" size="1.016" layer="25" font="vector" ratio="15" rot="R90"/>
 </element>
 <element name="U$2" library="nickparts" package="ARACHNID_LABS_LOGO_SM" value="" x="5.08" y="7.62" rot="MR90"/>
-<element name="R2" library="SparkFun-Passives" package="0603-RES" value="60" x="22.225" y="8.89" smashed="yes">
-<attribute name="NAME" x="21.336" y="7.112" size="1.016" layer="25" font="vector" ratio="15"/>
-</element>
-<element name="C1" library="SparkFun-Capacitors" package="0603-CAP" value="" x="24.13" y="11.43" smashed="yes">
-<attribute name="NAME" x="22.479" y="11.938" size="1.016" layer="25" font="vector" ratio="15" rot="R180"/>
-<attribute name="VALUE" x="23.114" y="10.287" size="0.4064" layer="27" font="vector"/>
+<element name="R2" library="SparkFun-Passives" package="0603-RES" value="60" x="17.78" y="8.89" smashed="yes">
+<attribute name="NAME" x="16.891" y="7.112" size="1.016" layer="25" font="vector" ratio="15"/>
+</element>
+<element name="C1" library="SparkFun-Capacitors" package="0603-CAP" value="" x="19.685" y="11.43" smashed="yes">
+<attribute name="NAME" x="18.034" y="11.938" size="1.016" layer="25" font="vector" ratio="15" rot="R180"/>
+<attribute name="VALUE" x="18.669" y="10.287" size="0.4064" layer="27" font="vector"/>
 </element>
 </elements>
 <signals>
-<signal name="N$3">
+<signal name="N$4">
+<contactref element="C1" pad="2"/>
+<wire x1="20.535" y1="11.43" x2="24.605" y2="11.43" width="0.6096" layer="1"/>
 <contactref element="U$1" pad="8"/>
-<contactref element="J1" pad="PWR"/>
-<wire x1="19.05" y1="3.175" x2="22.495" y2="3.175" width="0.8128" layer="1"/>
-<wire x1="22.495" y1="3.175" x2="26.94" y2="7.62" width="0.8128" layer="1"/>
-</signal>
-<signal name="N$4">
-<contactref element="J1" pad="GNDBREAK"/>
 <contactref element="U$1" pad="7"/>
 <contactref element="J1" pad="GND"/>
-<wire x1="16.51" y1="4.445" x2="16.51" y2="2.54" width="0.8128" layer="16"/>
-<wire x1="16.51" y1="2.54" x2="17.78" y2="1.27" width="0.8128" layer="16"/>
-<wire x1="17.78" y1="1.27" x2="26.67" y2="1.27" width="0.8128" layer="16"/>
-<wire x1="26.67" y1="1.27" x2="33.02" y2="7.62" width="0.8128" layer="16"/>
-<wire x1="33.02" y1="7.62" x2="32.94" y2="7.62" width="0.8128" layer="16"/>
-<wire x1="29.94" y1="12.32" x2="29.94" y2="10.7" width="0.8128" layer="16"/>
-<wire x1="29.94" y1="10.7" x2="33.02" y2="7.62" width="0.8128" layer="16"/>
-<wire x1="33.02" y1="7.62" x2="32.94" y2="7.62" width="0.8128" layer="16"/>
-<contactref element="C1" pad="2"/>
-<wire x1="24.98" y1="11.43" x2="29.05" y2="11.43" width="0.6096" layer="1"/>
-<wire x1="29.05" y1="11.43" x2="29.94" y2="12.32" width="0.6096" layer="1"/>
+<contactref element="J1" pad="GNDBREAK"/>
+<wire x1="24.605" y1="11.43" x2="24.685" y2="11.51" width="0.6096" layer="1"/>
+<wire x1="24.685" y1="11.51" x2="25.495" y2="12.32" width="0.6096" layer="1"/>
+<wire x1="28.495" y1="7.62" x2="28.495" y2="7.7" width="0.6096" layer="1"/>
+<wire x1="28.495" y1="7.7" x2="24.685" y2="11.51" width="0.6096" layer="1"/>
+<wire x1="12.065" y1="4.445" x2="13.335" y2="4.445" width="0.6096" layer="1"/>
+<wire x1="13.335" y1="4.445" x2="14.605" y2="3.175" width="0.6096" layer="1"/>
+<wire x1="14.605" y1="3.175" x2="24.05" y2="3.175" width="0.6096" layer="1"/>
+<wire x1="24.05" y1="3.175" x2="28.495" y2="7.62" width="0.6096" layer="1"/>
 </signal>
 <signal name="N$1">
 <contactref element="U$1" pad="1"/>
 <contactref element="R1" pad="1"/>
-<wire x1="21.375" y1="13.97" x2="18.415" y2="13.97" width="0.6096" layer="1"/>
-<wire x1="18.415" y1="13.97" x2="16.51" y2="12.065" width="0.6096" layer="1"/>
+<wire x1="16.93" y1="13.97" x2="13.97" y2="13.97" width="0.6096" layer="1"/>
+<wire x1="13.97" y1="13.97" x2="12.065" y2="12.065" width="0.6096" layer="1"/>
 </signal>
 <signal name="N$2">
 <contactref element="U$1" pad="2"/>
 <contactref element="R2" pad="1"/>
-<wire x1="21.375" y1="8.89" x2="20.955" y2="8.89" width="0.6096" layer="1"/>
-<wire x1="20.955" y1="8.89" x2="19.05" y2="10.795" width="0.6096" layer="1"/>
+<wire x1="16.93" y1="8.89" x2="16.51" y2="8.89" width="0.6096" layer="1"/>
+<wire x1="16.51" y1="8.89" x2="14.605" y2="10.795" width="0.6096" layer="1"/>
 </signal>
 <signal name="N$5">
@@
 <contactref element="C1" pad="1"/>
 <contactref element="R1" pad="2"/>
-<wire x1="23.075" y1="13.97" x2="23.075" y2="11.635" width="0.6096" layer="1"/>
-<wire x1="23.075" y1="11.635" x2="23.28" y2="11.43" width="0.6096" layer="1"/>
-<wire x1="23.075" y1="8.89" x2="23.075" y2="11.225" width="0.6096" layer="1"/>
-<wire x1="23.075" y1="11.225" x2="23.28" y2="11.43" width="0.6096" layer="1"/>
+<wire x1="18.63" y1="13.97" x2="18.63" y2="11.635" width="0.6096" layer="1"/>
+<wire x1="18.63" y1="11.635" x2="18.835" y2="11.43" width="0.6096" layer="1"/>
+<wire x1="18.63" y1="8.89" x2="18.63" y2="11.225" width="0.6096" layer="1"/>
+<wire x1="18.63" y1="11.225" x2="18.835" y2="11.43" width="0.6096" layer="1"/>
+</signal>
+<signal name="N$3">
+<contactref element="J1" pad="PWR"/>
+<contactref element="U$1" pad="5"/>
+<contactref element="U$1" pad="4"/>
+<wire x1="12.065" y1="6.985" x2="13.335" y2="6.985" width="0.6096" layer="16"/>
+<wire x1="13.335" y1="6.985" x2="14.605" y2="8.255" width="0.6096" layer="16"/>
+<wire x1="14.605" y1="8.255" x2="15.24" y2="8.255" width="0.6096" layer="16"/>
+<wire x1="15.24" y1="8.255" x2="15.875" y2="7.62" width="0.6096" layer="16"/>
+<wire x1="15.875" y1="7.62" x2="22.495" y2="7.62" width="0.6096" layer="16"/>
 </signal>
 </signals>
