File: shield/shield.brd (EAGLE design)
At the start: 68.6 x 53.3 mm, 25 parts, among them IC1 MCP2515-E/SO, IC2 MCP2562, IC3 LM2595NDH

Commit message: Added TVS diodes, fixed silkscreen issues
Parts:
- added IC4: PESD1CAN, nickparts:SOT23
Connections:
- net CANH: now also IC4.1
- net CANL: now also IC4.2
- net GND: now also IC4.3
Routing:
- net GND: track 221.0 -> 224.6 mm, vias 8 -> 9
- net CANL: track 39.1 -> 42.0 mm
- net CANH: track 48.3 -> 51.2 mm
- net V+: track 111.9 -> 112.8 mm
Changed lines of the file:
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@@
 <elements>
 <element name="IC3" library="nickparts" package="TO263-5" value="LM2595NDH" x="40.64" y="13.97" smashed="yes" rot="R180">
-<attribute name="NAME" x="41.783" y="14.097" size="1.016" layer="25" font="vector" ratio="15" rot="R180"/>
+<attribute name="NAME" x="43.688" y="22.352" size="1.016" layer="25" font="vector" ratio="15" rot="R180"/>
 </element>
 <element name="C3" library="SparkFun-Capacitors" package="PANASONIC_G" value="" x="37.465" y="27.305" smashed="yes" rot="R270">
@@
 <element name="U$5" library="SparkFun-Aesthetics" package="OSHW-LOGO-M" value="" x="26.035" y="28.575"/>
 <element name="C7" library="SparkFun-Passives" package="0603-CAP" value="0.1u" x="25.4" y="15.24" rot="R90"/>
-<element name="S1" library="SparkFun-Electromechanical" package="AYZ0202" value="DPDT" x="16.51" y="38.1" rot="R90">
+<element name="S1" library="SparkFun-Electromechanical" package="AYZ0202" value="DPDT" x="16.51" y="38.1" smashed="yes" rot="R90">
 <attribute name="PROD_ID" value="SWCH-08179" x="16.51" y="38.1" size="1.778" layer="27" rot="R90" display="off"/>
+<attribute name="NAME" x="16.51" y="35.687" size="1.016" layer="25" font="vector" ratio="15" rot="R180" align="bottom-center"/>
 </element>
 <element name="R2" library="SparkFun-Passives" package="0603-RES" value="60" x="19.05" y="43.815" smashed="yes" rot="R270">
@@
 <element name="C8" library="SparkFun-Passives" package="0603-CAP" value="4.7nF" x="16.51" y="43.815" smashed="yes" rot="R270">
 <attribute name="NAME" x="17.018" y="45.466" size="1.016" layer="25" font="vector" ratio="15" rot="R90"/>
+</element>
+<element name="IC4" library="nickparts" package="SOT23" value="PESD1CAN" x="29.21" y="8.89" smashed="yes" rot="R180">
+<attribute name="NAME" x="33.274" y="9.398" size="1.016" layer="25" font="vector" ratio="15" rot="R180"/>
 </element>
 </elements>
@@
 <via x="33.02" y="17.145" extent="1-16" drill="0.3"/>
 <wire x1="27.94" y1="5.08" x2="29.21" y2="6.35" width="0.508" layer="16"/>
-<wire x1="29.21" y1="6.35" x2="29.21" y2="12.7" width="0.508" layer="16"/>
+<wire x1="29.21" y1="6.35" x2="29.21" y2="8.89" width="0.508" layer="16"/>
+<wire x1="29.21" y1="8.89" x2="29.21" y2="12.7" width="0.508" layer="16"/>
 <wire x1="29.21" y1="12.7" x2="29.21" y2="16.51" width="0.508" layer="16"/>
 <wire x1="29.21" y1="16.51" x2="29.845" y2="17.145" width="0.508" layer="16"/>
@@
 <via x="16.51" y="41.91" extent="1-16" drill="0.3"/>
 <wire x1="16.51" y1="41.91" x2="26.416" y2="41.91" width="0.254" layer="16"/>
+<contactref element="IC4" pad="3"/>
+<wire x1="29.21" y1="7.79" x2="29.21" y2="8.89" width="0.4064" layer="1"/>
+<via x="29.21" y="8.89" extent="1-16" drill="0.3"/>
+<wire x1="29.21" y1="8.89" x2="29.21" y2="6.35" width="0.4064" layer="16"/>
 </signal>
 <signal name="N$6">
@@
 <wire x1="12.7" y1="37.465" x2="12.7" y2="31.115" width="0.254" layer="1"/>
 <wire x1="12.7" y1="31.115" x2="16.51" y2="27.305" width="0.254" layer="1"/>
+<contactref element="IC4" pad="1"/>
+<wire x1="30.16" y1="9.99" x2="29.845" y2="9.99" width="0.4064" layer="1"/>
+<wire x1="29.845" y1="9.99" x2="29.845" y2="12.6238" width="0.4064" layer="1"/>
 </signal>
 <signal name="CANL">
@@
 <wire x1="20.32" y1="37.465" x2="20.32" y2="27.305" width="0.254" layer="1"/>
 <wire x1="20.32" y1="27.305" x2="19.05" y2="26.035" width="0.254" layer="1"/>
+<contactref element="IC4" pad="2"/>
+<wire x1="28.26" y1="9.99" x2="28.575" y2="9.99" width="0.4064" layer="1"/>
+<wire x1="28.575" y1="9.99" x2="28.575" y2="12.6238" width="0.4064" layer="1"/>
 </signal>
 <signal name="VIN">
@@
 <wire x1="58.2422" y1="46.99" x2="59.69" y2="46.99" width="0.254" layer="1"/>
 <wire x1="59.69" y1="34.925" x2="54.19" y2="34.925" width="0.254" layer="1"/>
-<wire x1="27.305" y1="12.6238" x2="27.305" y2="7.62" width="0.254" layer="1"/>
-<wire x1="27.305" y1="7.62" x2="27.94" y2="6.985" width="0.254" layer="1"/>
-<wire x1="27.94" y1="6.985" x2="32.385" y2="6.985" width="0.254" layer="1"/>
 <via x="32.385" y="6.985" extent="1-16" drill="0.3"/>
 <wire x1="32.385" y1="6.985" x2="33.655" y2="6.985" width="0.254" layer="16"/>
@@
 <wire x1="61.595" y1="6.35" x2="61.595" y2="22.225" width="0.254" layer="1"/>
 <wire x1="61.595" y1="22.225" x2="61.2775" y2="22.5425" width="0.254" layer="1"/>
+<wire x1="27.305" y1="12.6238" x2="27.305" y2="6.985" width="0.254" layer="1"/>
+<wire x1="27.305" y1="6.985" x2="27.94" y2="6.35" width="0.254" layer="1"/>
+<wire x1="27.94" y1="6.35" x2="31.75" y2="6.35" width="0.254" layer="1"/>
+<wire x1="31.75" y1="6.35" x2="32.385" y2="6.985" width="0.254" layer="1"/>
 </signal>
 <signal name="N$7">

Commit message: Minor changes to shield, rpi board, and cape
Parts:
- removed L1: MSS1260, nickparts:MSS1260
- added C10: 56u, nickparts:SM_RADIAL_6.3AMM
- added C9: 10n, nickparts:0805
- added I1: SRN8040-330M, nickparts:SRN8040
- C3: value (none) -> 4.7u; device SparkFun-Capacitors:PANASONIC_G -> nickparts:1206
- C4: value (none) -> 1u; device SparkFun-Capacitors:PANASONIC_E -> nickparts:0805
- D1: value (none) -> B240A-13-F; device SparkFun-DiscreteSemi:SMA-DIODE_ALT -> nickparts:SMA
- IC3: value LM2595NDH -> LM22675MR-5.0/NOPB; device nickparts:TO263-5 -> nickparts:MRA08B
- U$1: value ARDUINO_R3_ICSP -> ARDUINO_R3_ICSPNODIM; device adafruit:ARDUINOR3_ICSP -> nickparts:ARDUINOR3_ICSP_NODIM
- moved C7 36.9 mm to (41.9, 48.3), turned to 0 degrees
- moved IC4 36.1 mm to (35.6, 44.5), turned to 90 degrees
- moved IC2 31.9 mm to (41.9, 44.5), turned to 90 degrees
- moved U$5 28.4 mm to (49.5, 12.7), turned to 270 degrees
- moved U$4 28.2 mm to (48.9, 20.3), turned to 270 degrees
- moved C6 26.9 mm to (41.9, 40.6), turned to 0 degrees
- moved C4 24.2 mm to (27.9, 20.3), turned to 90 degrees
- moved D1 21.5 mm to (24.8, 19.7), turned to 90 degrees
- moved C3 18.0 mm to (25.4, 14.0), turned to 0 degrees
- moved IC3 9.92 mm to (33.0, 20.3)
- moved C2 8.47 mm to (41.9, 33.7), turned to 270 degrees
- moved Y1 5.24 mm to (45.1, 33.7), turned to 270 degrees
- moved C1 4.84 mm to (48.3, 33.7), turned to 90 degrees
- moved U$2 4.45 mm to (5.71, 22.9)
- moved U$3 4.45 mm to (5.71, 7.62)
Connections:
- net N$1 renamed RXCAN
- removed net N$11: U$2.5, U$3.5
- removed net N$6: D1.C, IC3.1, L1.P$1
- new net N$9: U$2.3, U$3.3
- new net SWOUT: C9.2, D1.1, I1.2, IC3.8
- net +5V: now also C10.1, I1.1; no longer C4.+, L1.P$2
- net GND: now also C10.2, C3.2, C4.2, D1.2, IC3.EPAD, U$2.8, U$3.8; no longer C3.-, C4.-, D1.A, IC3.3, IC3.5, U$2.3, U$3.3
- net N$10: now also C9.1, IC3.1; no longer U$2.4, U$3.4
- net VCC: now also C3.1, C4.1, IC3.7, U$2.4, U$2.5, U$3.4, U$3.5; no longer C3.+, IC3.2, U$2.8, U$3.8
Routing:
- net RXCAN: track 56.8 -> 4.53 mm
- net TXCAN: track 51.5 -> 11.6 mm
- net V+: track 112.8 -> 75.7 mm, vias 4 -> 3
- net GND: track 224.6 -> 189.1 mm, vias 9 -> 18
- net CANL: track 42.0 -> 66.6 mm
- net CANH: track 51.2 -> 72.5 mm
- net N$11: track 19.5 -> 0.00 mm
- net N$9: track 0.00 -> 17.9 mm, vias 0 -> 1
- net N$6: track 16.1 -> 0.00 mm
- net SWOUT: track 0.00 -> 15.9 mm
- net N$10: track 18.4 -> 2.62 mm, vias 1 -> 0
- net +5V: track 122.2 -> 111.3 mm, vias 3 -> 4
- net VCC: track 62.2 -> 53.4 mm, vias 2 -> 0
- net N$5: track 5.43 -> 9.76 mm
- net N$8: track 17.9 -> 22.1 mm, vias 1 -> 0
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- added copper zone on layer 1, net SWOUT
- removed copper zone on layer 1, net N$6
- removed copper zone on layer 1, net VCC
Other:
- outline, holes or cut-outs redrawn
- board text added: "uCAN Arduino Shield v1.0.1"
- board text removed: "uCAN Arduino Shield v1.0"
